Commit message: Add PID tuning scripts and GUI for humanoid arm control
- Implemented a simple PID auto-tuning script (auto_tune_pid_simple.py) to facilitate tuning of joint controllers by iteratively adjusting P, I, and D gains based on system response.
- Enhanced the PID tuner GUI (pid_tuner_gui.py) to detect active controllers dynamically and display the current PID gains for selected joints.
- Introduced a new trajectory tuner UI (trajectory_tuner_ui.py) that allows users to send test trajectories and visualize joint position tracking and error.
- Added a Qt Designer UI file (trajectory_tuner.ui) for the trajectory tuner interface.
- Updated the URDF model to temporarily increase the effort limit for the shoulder joint to aid in PID tuning.

File: humanoid_arm_description/urdf/humanoid_arm_5dof_macro.urdf.xacro (robot description, xacro)
@@ -88,5 +88,6 @@
       <child link="${prefix}upper_arm_link"/>
       <axis xyz="1 0 0"/>
-      <limit lower="-3.14" upper="3.14" effort="120" velocity="3"/>
+      <!-- Temporarily increased for PID tuning - Real motor: 120 Nm -->
+      <limit lower="-3.14" upper="3.14" effort="500" velocity="3"/>
       <dynamics damping="0.1" friction="0.1"/>
     </joint>

Commit message: Add multiple scripts for reaching targets with different methods
- Implemented `reach_target_ik.py` using MoveIt2's IK solver for reaching specific XYZ coordinates and predefined targets.
- Created `reach_target_moveit.py` utilizing MoveIt's move_group action interface for simpler target reaching.
- Developed `reach_target_simple.py` to send joint trajectories directly to the joint_trajectory_controller without MoveIt2.
- Added `reach_with_ik.py` to compute IK using the /compute_ik service and execute the trajectory.
- Updated URDF to include a world link and fixed joint for grounding in Gazebo.
- Adjusted joint limits in MoveIt configuration for higher velocity and acceleration scaling factors.
- Enhanced move_group simulation launch file with increased tolerances for trajectory execution.

File: humanoid_arm_description/urdf/humanoid_arm_5dof_macro.urdf.xacro (robot description, xacro)
@@ -13,4 +13,12 @@
   <!-- Robot macro -->
   <xacro:macro name="humanoid_arm_5dof_macro" params="prefix use_fake_hardware:=true fake_sensor_commands:=false slowdown:=3.0 robot_controller:=joint_trajectory_controller">
+    <!-- World link (massless, for fixing base to world in Gazebo) -->
+    <link name="${prefix}world"/>
+    <!-- Fixed joint: world -> base_link (fixes base to ground) -->
+    <joint name="${prefix}world_to_base_joint" type="fixed">
+      <parent link="${prefix}world"/>
+      <child link="${prefix}base_link"/>
+      <origin xyz="0 0 0" rpy="0 0 0"/>
+    </joint>
     <!-- Base Link -->
     <link name="${prefix}base_link">
