Commit message: Add PID tuning guide, update Gazebo launch, and modify controller configurations
- Introduced a comprehensive PID tuning guide in PID_README.md for the humanoid arm's joint trajectory controller, detailing tools, methods, and workflows for effective tuning.
- Updated the Gazebo launch file to use the new ros_gz_sim package, simplifying the launch process and removing the need for a separate control node.
- Changed the joint trajectory controller configuration in controllers.yaml to use effort control instead of position, and adjusted constraints for better performance.
- Enhanced the test trajectory script to include current joint position retrieval and PID gain display, improving usability during testing.
- Modified the URDF files to include effort command interfaces for all joints, ensuring compatibility with the new control strategy.
- Adjusted dynamics parameters in the URDF to reduce damping and friction, allowing for more responsive joint movements.

File: humanoid_arm_description/urdf/humanoid_arm_5dof.ros2_control.xacro (robot description, xacro)
@@ -25,4 +25,8 @@
           <param name="max">3.0</param>
         </command_interface>
+        <command_interface name="effort">
+          <param name="min">-120.0</param>
+          <param name="max">120.0</param>
+        </command_interface>
         <state_interface name="position">
           <param name="initial_value">0.0</param>
@@ -40,4 +44,8 @@
           <param name="min">-3.0</param>
           <param name="max">3.0</param>
+        </command_interface>
+        <command_interface name="effort">
+          <param name="min">-120.0</param>
+          <param name="max">120.0</param>
         </command_interface>
         <state_interface name="position">
@@ -57,4 +65,8 @@
           <param name="max">1.6</param>
         </command_interface>
+        <command_interface name="effort">
+          <param name="min">-60.0</param>
+          <param name="max">60.0</param>
+        </command_interface>
         <state_interface name="position">
           <param name="initial_value">0.0</param>
@@ -73,4 +85,8 @@
           <param name="max">1.6</param>
         </command_interface>
+        <command_interface name="effort">
+          <param name="min">-60.0</param>
+          <param name="max">60.0</param>
+        </command_interface>
         <state_interface name="position">
           <param name="initial_value">0.0</param>
@@ -88,4 +104,8 @@
           <param name="min">-0.8</param>
           <param name="max">0.8</param>
+        </command_interface>
+        <command_interface name="effort">
+          <param name="min">-17.0</param>
+          <param name="max">17.0</param>
         </command_interface>
         <state_interface name="position">

File: humanoid_arm_description/urdf/humanoid_arm_5dof_macro.urdf.xacro (robot description, xacro)
@@ -89,5 +89,5 @@
       <axis xyz="1 0 0"/>
       <limit lower="-3.14" upper="3.14" effort="120" velocity="3"/>
-      <dynamics damping="0.7" friction="0.5"/>
+      <dynamics damping="0.1" friction="0.1"/>
     </joint>
     <!-- Shoulder Pitch Motor Link -->
@@ -119,5 +119,5 @@
       <axis xyz="0 1 0"/>
       <limit lower="-0.55" upper="3.1" effort="120" velocity="3"/>
-      <dynamics damping="0.7" friction="0.5"/>
+      <dynamics damping="0.1" friction="0.1"/>
     </joint>
     <!-- Forearm Link -->
@@ -203,5 +203,5 @@
       <axis xyz="-0.209 0 -0.978"/>
       <limit lower="-3.14" upper="3.14" effort="60" velocity="1.6"/>
-      <dynamics damping="0.5" friction="0.3"/>
+      <dynamics damping="0.1" friction="0.1"/>
     </joint>
     <!-- Wrist Base Link -->
@@ -287,5 +287,5 @@
       <axis xyz="-1 0 0"/>
       <limit lower="-0.31" upper="2.8" effort="60" velocity="1.6"/>
-      <dynamics damping="0.5" friction="0.3"/>
+      <dynamics damping="0.1" friction="0.1"/>
     </joint>
     <!-- Wrist Assembly Link -->
@@ -371,5 +371,5 @@
       <axis xyz="0 -1 0"/>
       <limit lower="-3.14" upper="3.14" effort="17" velocity="0.8"/>
-      <dynamics damping="0.3" friction="0.2"/>
+      <dynamics damping="0.1" friction="0.1"/>
     </joint>
     <!-- End Motor Link (Optional - for completeness) -->

Commit message: Fixed Actuator specs with corect Robstride datasheet, speeds, loads and timings Add trajectory timing documentation and enhance actuator specifications - Introduced a comprehensive `TRAJECTORY_TIMING.md` document detailing the `time_from_start` parameter, speed-time tradeoffs, and optimal timing calculations for trajectory controllers in ROS2. - Updated `actuator_specs.yaml` to reflect new motor specifications, including torque, speed, and electrical characteristics for various joints. - Modified `joint_control.py` to implement a fixed response time for joint commands, improving responsiveness. - Enhanced URDF files to load actuator specifications dynamically, ensuring joint limits are based on actual motor capabilities. - Adjusted `joint_limits.yaml` to align with updated actuator specifications, increasing velocity and acceleration limits for improved performance.

File: humanoid_arm_description/urdf/humanoid_arm_5dof.ros2_control.xacro (robot description, xacro)
@@ -1,4 +1,6 @@
 <?xml version="1.0"?>
 <robot xmlns:xacro="http://www.ros.org/wiki/xacro">
+  <!-- Load actuator specifications from YAML -->
+  <xacro:property name="actuator_specs" value="${xacro.load_yaml('$(find humanoid_arm_control)/config/actuator_specs.yaml')}" />
   <xacro:macro name="humanoid_arm_5dof_ros2_control" params="name prefix use_fake_hardware:=true fake_sensor_commands:=false slowdown:=3.0 robot_controller:=joint_trajectory_controller">
     <ros2_control name="${name}" type="system">
@@ -22,10 +24,10 @@
         </command_interface>
         <command_interface name="velocity">
-          <param name="min">-3.0</param>
-          <param name="max">3.0</param>
+          <param name="min">-${actuator_specs['actuators']['base_rotation_joint']['motor']['max_speed']}</param>
+          <param name="max">${actuator_specs['actuators']['base_rotation_joint']['motor']['max_speed']}</param>
         </command_interface>
         <command_interface name="effort">
-          <param name="min">-120.0</param>
-          <param name="max">120.0</param>
+          <param name="min">-${actuator_specs['actuators']['base_rotation_joint']['motor']['max_torque']}</param>
+          <param name="max">${actuator_specs['actuators']['base_rotation_joint']['motor']['max_torque']}</param>
         </command_interface>
         <state_interface name="position">
@@ -42,10 +44,10 @@
         </command_interface>
         <command_interface name="velocity">
-          <param name="min">-3.0</param>
-          <param name="max">3.0</param>
+          <param name="min">-${actuator_specs['actuators']['shoulder_pitch_joint']['motor']['max_speed']}</param>
+          <param name="max">${actuator_specs['actuators']['shoulder_pitch_joint']['motor']['max_speed']}</param>
         </command_interface>
         <command_interface name="effort">
-          <param name="min">-120.0</param>
-          <param name="max">120.0</param>
+          <param name="min">-${actuator_specs['actuators']['shoulder_pitch_joint']['motor']['max_torque']}</param>
+          <param name="max">${actuator_specs['actuators']['shoulder_pitch_joint']['motor']['max_torque']}</param>
         </command_interface>
         <state_interface name="position">
@@ -62,10 +64,10 @@
         </command_interface>
         <command_interface name="velocity">
-          <param name="min">-1.6</param>
-          <param name="max">1.6</param>
+          <param name="min">-${actuator_specs['actuators']['elbow_pitch_joint']['motor']['max_speed']}</param>
+          <param name="max">${actuator_specs['actuators']['elbow_pitch_joint']['motor']['max_speed']}</param>
         </command_interface>
         <command_interface name="effort">
-          <param name="min">-60.0</param>
-          <param name="max">60.0</param>
+          <param name="min">-${actuator_specs['actuators']['elbow_pitch_joint']['motor']['max_torque']}</param>
+          <param name="max">${actuator_specs['actuators']['elbow_pitch_joint']['motor']['max_torque']}</param>
         </command_interface>
         <state_interface name="position">
@@ -82,10 +84,10 @@
         </command_interface>
         <command_interface name="velocity">
-          <param name="min">-1.6</param>
-          <param name="max">1.6</param>
+          <param name="min">-${actuator_specs['actuators']['wrist_pitch_joint']['motor']['max_speed']}</param>
+          <param name="max">${actuator_specs['actuators']['wrist_pitch_joint']['motor']['max_speed']}</param>
         </command_interface>
         <command_interface name="effort">
-          <param name="min">-60.0</param>
-          <param name="max">60.0</param>
+          <param name="min">-${actuator_specs['actuators']['wrist_pitch_joint']['motor']['max_torque']}</param>
+          <param name="max">${actuator_specs['actuators']['wrist_pitch_joint']['motor']['max_torque']}</param>
         </command_interface>
         <state_interface name="position">
@@ -102,10 +104,10 @@
         </command_interface>
         <command_interface name="velocity">
-          <param name="min">-0.8</param>
-          <param name="max">0.8</param>
+          <param name="min">-${actuator_specs['actuators']['wrist_roll_joint']['motor']['max_speed']}</param>
+          <param name="max">${actuator_specs['actuators']['wrist_roll_joint']['motor']['max_speed']}</param>
         </command_interface>
         <command_interface name="effort">
-          <param name="min">-17.0</param>
-          <param name="max">17.0</param>
+          <param name="min">-${actuator_specs['actuators']['wrist_roll_joint']['motor']['max_torque']}</param>
+          <param name="max">${actuator_specs['actuators']['wrist_roll_joint']['motor']['max_torque']}</param>
         </command_interface>
         <state_interface name="position">

File: humanoid_arm_description/urdf/humanoid_arm_5dof_macro.urdf.xacro (robot description, xacro)
@@ -1,4 +1,6 @@
 <?xml version="1.0"?>
 <robot xmlns:xacro="http://www.ros.org/wiki/xacro">
+  <!-- Load actuator specifications from YAML -->
+  <xacro:property name="actuator_specs" value="${xacro.load_yaml('$(find humanoid_arm_control)/config/actuator_specs.yaml')}" />
   <!-- Materials -->
   <material name="base_material">
@@ -96,6 +98,8 @@
       <child link="${prefix}upper_arm_link"/>
       <axis xyz="1 0 0"/>
-      <!-- Temporarily increased for PID tuning - Real motor: 120 Nm -->
-      <limit lower="-3.14" upper="3.14" effort="500" velocity="3"/>
+      <!-- Loaded from actuator_specs.yaml -->
+      <limit lower="-3.14" upper="3.14"
+             effort="${actuator_specs['actuators']['base_rotation_joint']['motor']['max_torque']}"
+             velocity="${actuator_specs['actuators']['base_rotation_joint']['motor']['max_speed']}"/>
       <dynamics damping="0.1" friction="0.1"/>
     </joint>
@@ -127,5 +131,8 @@
       <child link="${prefix}shoulder_pitch_motor_link"/>
       <axis xyz="0 1 0"/>
-      <limit lower="-0.55" upper="3.1" effort="120" velocity="3"/>
+      <!-- Loaded from actuator_specs.yaml -->
+      <limit lower="-0.55" upper="3.1"
+             effort="${actuator_specs['actuators']['shoulder_pitch_joint']['motor']['max_torque']}"
+             velocity="${actuator_specs['actuators']['shoulder_pitch_joint']['motor']['max_speed']}"/>
       <dynamics damping="0.1" friction="0.1"/>
     </joint>
@@ -211,5 +218,8 @@
       <child link="${prefix}elbow_flange_link"/>
       <axis xyz="-0.209 0 -0.978"/>
-      <limit lower="-3.14" upper="3.14" effort="60" velocity="1.6"/>
+      <!-- Loaded from actuator_specs.yaml -->
+      <limit lower="-3.14" upper="3.14"
+             effort="${actuator_specs['actuators']['elbow_pitch_joint']['motor']['max_torque']}"
+             velocity="${actuator_specs['actuators']['elbow_pitch_joint']['motor']['max_speed']}"/>
       <dynamics damping="0.1" friction="0.1"/>
     </joint>
@@ -295,5 +305,8 @@
       <child link="${prefix}wrist_pitch_link"/>
       <axis xyz="-1 0 0"/>
-      <limit lower="-0.31" upper="2.8" effort="60" velocity="1.6"/>
+      <!-- Loaded from actuator_specs.yaml -->
+      <limit lower="-0.31" upper="2.8"
+             effort="${actuator_specs['actuators']['wrist_pitch_joint']['motor']['max_torque']}"
+             velocity="${actuator_specs['actuators']['wrist_pitch_joint']['motor']['max_speed']}"/>
       <dynamics damping="0.1" friction="0.1"/>
     </joint>
@@ -379,5 +392,8 @@
       <child link="${prefix}end_effector_link"/>
       <axis xyz="0 -1 0"/>
-      <limit lower="-3.14" upper="3.14" effort="17" velocity="0.8"/>
+      <!-- Loaded from actuator_specs.yaml -->
+      <limit lower="-3.14" upper="3.14"
+             effort="${actuator_specs['actuators']['wrist_roll_joint']['motor']['max_torque']}"
+             velocity="${actuator_specs['actuators']['wrist_roll_joint']['motor']['max_speed']}"/>
       <dynamics damping="0.1" friction="0.1"/>
     </joint>
